File: PCB/A4/A4_STEPPERS.sch (KiCad schematic (older format))
At the start: 40 parts, among them J10 Conn_02x03_Odd_Even, J11 Conn_01x04_Male, J12 Conn_01x04_Male, J14 Conn_01x02_Male, J16 Conn_01x02_Male, J17 Conn_01x06_Male, J18 Conn_01x06_Male, J19 Conn_02x03_Odd_Even, J20 Conn_02x03_Odd_Even, J21 Conn_01x04_Male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

Commit message: PCB ready to order
Connections:
- net ENC1 renamed ENC1A
Changed lines of the file:
@@
 $EndComp
 Text GLabel 8250 2600 2    50   Input ~ 0
-ENC1
+ENC1A
 $Comp
 L power:+3V3 #PWR?
