File: PCBs/A4/A4.sch (KiCad schematic (older format))
At the start: 40 parts, among them J1 Barrel_Jack_Switch, J13 Conn_01x06_Male, J15 Conn_01x06_Male, J2 Conn_01x02_Male, J25 Conn_01x04_Male, J3 Conn_01x06_Male, J4 Conn_01x02_Male, J7 Screw_Terminal_01x02, J8 Screw_Terminal_01x02, Q1 2N7002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

Commit message: 5 stepper board
Parts:
- added J?: Screw_Terminal_01x02, TerminalBlock_Phoenix:TerminalBlock_Phoenix_MKDS-1,5-2_1x02_P5.00mm_Horizontal, symbol Connector:Screw_Terminal_01x02
Connections:
- net +12V: now also J?.1 (Pin_1)
- net GND: now also J?.2 (Pin_2)
Changed lines of the file:
@@
 Wire Wire Line
 	5650 3150 5650 3450
+$Comp
+L Connector:Screw_Terminal_01x02 J?
+U 1 1 6110BFC1
+P 1700 1500
+F 0 "J?" H 1780 1492 50  0000 L CNN
+F 1 "Screw_Terminal_01x02" H 1780 1401 50  0000 L CNN
+F 2 "TerminalBlock_Phoenix:TerminalBlock_Phoenix_MKDS-1,5-2_1x02_P5.00mm_Horizontal" H 1700 1500 50  0001 C CNN
+F 3 "~" H 1700 1500 50  0001 C CNN
+	1    1700 1500
+	1    0    0    -1
+$EndComp
+Wire Wire Line
+	1150 1500 1500 1500
+Connection ~ 1150 1500
+Wire Wire Line
+	1500 1600 1500 2100
+Wire Wire Line
+	1500 2100 1150 2100
+Connection ~ 1150 2100
 $EndSCHEMATC
